File: ASD2002.brd (EAGLE design)
At the start: 22.5 x 22.5 mm, 34 parts, among them J1 DF12-32-DS, J10 PIN_1X.1", J11 PIN_1X.1", J12 PIN_1X.1", J13 PIN_1X.1", J14 PIN_1X.1", J15 PIN_1X.1", J16 PIN_1X.1", J17 PIN_1X.1", J18 PIN_1X.1", J19 PIN_1X.1", J2 PIN_1X.1", J20 PIN_1X.1", J21 PIN_1X.1", J22 PIN_1X.1", J23 PIN_1X.1", J24 PIN_1X.1", J25 PIN_1X.1", J26 PIN_1X.1", J27 PIN_1X.1", J28 PIN_1X.1", J29 PIN_1X.1", J3 PIN_1X.1", J30 PIN_1X.1", J31 PIN_1X.1", J32 PIN_1X.1", J33 PIN_1X.1", J4 PIN_1X.1", J5 PIN_1X.1", J6 PIN_1X.1", J7 PIN_1X.1", J8 PIN_1X.1", J9 PIN_1X.1"

Commit message: Updated to Rev4
Routing:
- net VCC: track 14.1 -> 14.8 mm, vias 0 -> 2
- net IO3: track 15.9 -> 15.8 mm, vias 0 -> 2
Other:
- board text added: "0"
- board text added: "1"
- board text added: "10"
- board text added: "11"
- board text added: "12"
- board text added: "13"
- board text added: "2"
- board text added: "4"
- board text added: "5"
- board text added: "6"
- board text added: "7"
- board text added: "8"
- board text added: "9"
- board text added: "A0"
- board text added: "A1"
- board text added: "A2"
- board text added: "A3"
- board text added: "A4"
- board text added: "A5"
- board text added: "REV 4"
- board text removed: "AD0"
- board text removed: "AD1"
- board text removed: "AD2"
- board text removed: "AD3"
- board text removed: "AD4"
- board text removed: "AD5"
- board text removed: "IO0"
- board text removed: "IO1"
- board text removed: "IO2"
- board text removed: "IO3"
- board text removed: "IO4"
- board text removed: "IO5"
- board text removed: "IO6"
- board text removed: "IO7"
- board text removed: "IO8"
- board text removed: "IO9"
- board text removed: "MISO"
- board text removed: "MOSI"
- board text removed: "REV 3"
- board text removed: "SCK"
- board text removed: "SS"
